Commit message: Removed additional unnecessary .urdf and .xacro files. At this level: launch ==> gen3.xacro ==> gen3_macro.xacro & robotiq_2f_85_macro.xacro

File: kortex_description/robots/gen3.xacro (robot description, xacro)
@@ -5,4 +5,5 @@
     <xacro:arg name="dof" default="" />
     <xacro:arg name="vision" default="false" />
+    <xacro:arg name="parent" default="world" />
     <xacro:arg name="robot_ip" default="192.168.11.11" />
     <xacro:arg name="username" default="admin" />
@@ -24,36 +25,69 @@
     <xacro:arg name="use_internal_bus_gripper_comm" default="false" />
     <xacro:arg name="use_external_cable" default="false" />
-    <xacro:include filename="$(find kortex_description)/robots/kortex_robot.xacro" />
-    <!-- initial position for simulations (Mock Hardware, Gazebo, Ignition) -->
-    <xacro:arg name="initial_positions_file" default="$(find kortex_description)/config/initial_positions.yaml"/>
-    <!-- convert to property to use substitution in function -->
-    <xacro:property name="initial_positions_file" default="$(arg initial_positions_file)"/>
+    <xacro:arg name="initial_positions" default="${dict(joint_1=0.0,joint_2=0.0,joint_3=0.0,joint_4=0.0,joint_5=0.0,joint_6=0.0,joint_7=0.0)}"/>
+    <xacro:arg name="moveit_active" default="false" />
+    <xacro:arg name="gripper_com_port" default="/dev/ttyUSB0" />
+    <xacro:arg name="isaac_joint_commands" default="/isaac_joint_commands" />
+    <xacro:arg name="isaac_joint_states" default="/isaac_joint_states" />
+    <!-- Define world link -->
     <link name="world" />
-    <xacro:load_robot
-        parent="world"
-        arm="$(arg arm)"
-        gripper="$(arg gripper)"
-        gripper_joint_name="$(arg gripper_joint_name)"
-        gripper_max_velocity="$(arg gripper_max_velocity)"
-        gripper_max_force="$(arg gripper_max_force)"
-        dof="$(arg dof)"
-        vision="$(arg vision)"
-        robot_ip="$(arg robot_ip)"
-        username="$(arg username)"
-        password="$(arg password)"
-        port="$(arg port)"
-        port_realtime="$(arg port_realtime)"
-        session_inactivity_timeout_ms="$(arg session_inactivity_timeout_ms)"
-        connection_inactivity_timeout_ms="$(arg connection_inactivity_timeout_ms)"
-        use_internal_bus_gripper_comm="$(arg use_internal_bus_gripper_comm)"
-        prefix="$(arg prefix)"
-        use_fake_hardware="$(arg use_fake_hardware)"
-        fake_sensor_commands="$(arg fake_sensor_commands)"
-        sim_gazebo="$(arg sim_gazebo)"
-        sim_ignition="$(arg sim_ignition)"
-        sim_isaac="$(arg sim_isaac)"
-        use_external_cable="$(arg use_external_cable)"
-        initial_positions="${xacro.load_yaml(initial_positions_file)}" >
-        <origin xyz="0 0 0" rpy="0 0 0" />  <!-- position robot in the world -->
-    </xacro:load_robot>
+    <!-- Include and load arm macro files -->
+    <xacro:include filename="$(find kortex_description)/gen3_arm/urdf/${arm}_macro.xacro" />
+    <!-- Load the arm -->
+    <xacro:load_arm
+      parent="${parent}"
+      dof="${dof}"
+      vision="${vision}"
+      robot_ip="${robot_ip}"
+      username="${username}"
+      password="${password}"
+      port="${port}"
+      port_realtime="${port_realtime}"
+      session_inactivity_timeout_ms="${session_inactivity_timeout_ms}"
+      connection_inactivity_timeout_ms="${connection_inactivity_timeout_ms}"
+      prefix="${prefix}"
+      use_internal_bus_gripper_comm="${use_internal_bus_gripper_comm}"
+      use_fake_hardware="${use_fake_hardware}"
+      fake_sensor_commands="${fake_sensor_commands}"
+      sim_gazebo="${sim_gazebo}"
+      sim_ignition="${sim_ignition}"
+      sim_isaac="${sim_isaac}"
+      isaac_joint_commands="${isaac_joint_commands}"
+      isaac_joint_states="${isaac_joint_states}"
+      gripper_joint_name="${gripper_joint_name}"
+      gripper_max_velocity="${gripper_max_velocity}"
+      gripper_max_force="${gripper_max_force}"
+      use_external_cable="${use_external_cable}"
+      initial_positions="${initial_positions}"
+      moveit_active="${moveit_active}">
+      <origin xyz="0 0 0" rpy="0 0 0" />  <!-- position the robotic arm in the world -->
+    </xacro:load_arm>
+    <!-- If no gripper, define tool frame here -->
+    <xacro:if value="${not gripper}">
+      <link name="${prefix}tool_frame"/>
+      <joint name="${prefix}tool_frame_joint" type="fixed">
+        <origin xyz="0 0 0" rpy="0 0 0" />
+        <parent link="${prefix}${last_arm_link}" />
+        <child link="${prefix}tool_frame" />
+        <axis xyz="0 0 0" />
+      </joint>
+    </xacro:if>
+    <!-- Include and load the gripper if defined -->
+    <xacro:unless value="${not gripper}">
+      <xacro:include filename="$(find kortex_description)/gripper_robotiq_2f_85/urdf/${gripper}_macro.xacro" />
+      <!-- last_arm_link is defined in "$(find kortex_description)/arms/${arm}/urdf/${arm}_macro.xacro" -->
+      <xacro:load_gripper
+        parent="${prefix}${last_arm_link}"
+        prefix="${prefix}"
+        use_fake_hardware="${use_fake_hardware}"
+        fake_sensor_commands="${fake_sensor_commands}"
+        sim_ignition="${sim_ignition}"
+        sim_isaac="${sim_isaac}"
+        isaac_joint_commands="${isaac_joint_commands}"
+        isaac_joint_states="${isaac_joint_states}"
+        com_port="${gripper_com_port}"
+        use_internal_bus_gripper_comm="${use_internal_bus_gripper_comm}"
+        moveit_active="${moveit_active}"/>
+    </xacro:unless>
+  </xacro:macro>
 </robot>
