Commit message: Removed all the simulation related args/params from the .xacro files along with other unnecessary args/params

File: kortex_description/gen3_arm/urdf/gen3_macro.xacro (robot description, xacro)
@@ -5,42 +5,25 @@
   <xacro:property name="PI" value="3.1415926535897931"/>
   <xacro:macro name="load_arm" params="
-    parent
-    dof
-    vision
-    prefix
+    parent:=world
+    vision:=false
+    prefix:=""
     *origin
-    robot_ip
+    robot_ip:=192.168.1.10
     username:=admin
     password:=admin
     port:=10000
     port_realtime:=10001
-    session_inactivity_timeout_ms:=6000
+    session_inactivity_timeout_ms:=60000
     connection_inactivity_timeout_ms:=2000
-    use_internal_bus_gripper_comm:=true
-    gripper_joint_name
-    gripper_max_velocity:=100.0
-    gripper_max_force:=100.0
-    use_fake_hardware:=false
-    fake_sensor_commands:=false
-    sim_gazebo:=false
-    sim_ignition:=false
-    sim_isaac:=false
-    isaac_joint_commands:=/isaac_joint_commands
-    isaac_joint_states:=/isaac_joint_states
+    use_internal_bus_gripper_comm:=false
+    gripper_joint_name:=finger_joint
+    gripper_max_velocity:=100
+    gripper_max_force:=100
     use_external_cable:=false
-    initial_positions:=${dict(joint_1=0.0,joint_2=0.0,joint_3=0.0,joint_4=0.0,joint_5=0.0,joint_6=0.0,joint_7=0.0)}
-    moveit_active:=false">
+    initial_positions:=${dict(joint_1=0.0,joint_2=0.0,joint_3=0.0,joint_4=0.0,joint_5=0.0,joint_6=0.0,joint_7=0.0)}">
     <!-- ros2 control include -->
-    <xacro:include filename="$(find kortex_description)/arms/gen3/${dof}dof/urdf/kortex.ros2_control.xacro" />
+    <xacro:include filename="$(find kortex_description)/gen3_arm/urdf/kortex.ros2_control.xacro" />
     <xacro:kortex_ros2_control
       name="${prefix}KortexMultiInterfaceHardware" prefix="${prefix}"
-      use_fake_hardware="${use_fake_hardware}"
-      fake_sensor_commands="${fake_sensor_commands}"
-      sim_gazebo="${sim_gazebo}"
-      sim_ignition="${sim_ignition}"
-      sim_isaac="${sim_isaac}"
-      isaac_joint_commands="${isaac_joint_commands}"
-      isaac_joint_states="${isaac_joint_states}"
-      tf_prefix=""
       initial_positions="${initial_positions}"
       robot_ip="${robot_ip}"
@@ -69,14 +52,14 @@
         <origin xyz="0 0 0" rpy="0 0 0" />
         <geometry>
-          <mesh filename="file://$(find kortex_description)/arms/gen3/${dof}dof/meshes/base_link.dae" />
-        </geometry>
-        <material name="">
-          <color rgba="0.75294 0.75294 0.75294 1" />
-        </material>
-      </visual>
-      <collision>
-        <origin xyz="0 0 0" rpy="0 0 0" />
-        <geometry>
-          <mesh filename="file://$(find kortex_description)/arms/gen3/${dof}dof/meshes/base_link.dae" />
+          <mesh filename="file://$(find kortex_description)/gen3_arm/meshes/base_link.dae" />
+        </geometry>
+        <material name="">
+          <color rgba="0.75294 0.75294 0.75294 1" />
+        </material>
+      </visual>
+      <collision>
+        <origin xyz="0 0 0" rpy="0 0 0" />
+        <geometry>
+          <mesh filename="file://$(find kortex_description)/gen3_arm/meshes/base_link.dae" />
         </geometry>
       </collision>
@@ -91,14 +74,14 @@
         <origin xyz="0 0 0" rpy="0 0 0" />
         <geometry>
-          <mesh filename="file://$(find kortex_description)/arms/gen3/${dof}dof/meshes/shoulder_link.dae" />
-        </geometry>
-        <material name="">
-          <color rgba="0.75294 0.75294 0.75294 1" />
-        </material>
-      </visual>
-      <collision>
-        <origin xyz="0 0 0" rpy="0 0 0" />
-        <geometry>
-          <mesh filename="file://$(find kortex_description)/arms/gen3/${dof}dof/meshes/shoulder_link.dae" />
+          <mesh filename="file://$(find kortex_description)/gen3_arm/meshes/shoulder_link.dae" />
+        </geometry>
+        <material name="">
+          <color rgba="0.75294 0.75294 0.75294 1" />
+        </material>
+      </visual>
+      <collision>
+        <origin xyz="0 0 0" rpy="0 0 0" />
+        <geometry>
+          <mesh filename="file://$(find kortex_description)/gen3_arm/meshes/shoulder_link.dae" />
         </geometry>
       </collision>
@@ -147,14 +130,14 @@
         <origin xyz="0 0 0" rpy="0 0 0" />
         <geometry>
-          <mesh filename="file://$(find kortex_description)/arms/gen3/${dof}dof/meshes/half_arm_1_link.dae" />
-        </geometry>
-        <material name="">
-          <color rgba="0.75294 0.75294 0.75294 1" />
-        </material>
-      </visual>
-      <collision>
-        <origin xyz="0 0 0" rpy="0 0 0" />
-        <geometry>
-          <mesh filename="file://$(find kortex_description)/arms/gen3/${dof}dof/meshes/half_arm_1_link.dae" />
+          <mesh filename="file://$(find kortex_description)/gen3_arm/meshes/half_arm_1_link.dae" />
+        </geometry>
+        <material name="">
+          <color rgba="0.75294 0.75294 0.75294 1" />
+        </material>
+      </visual>
+      <collision>
+        <origin xyz="0 0 0" rpy="0 0 0" />
+        <geometry>
+          <mesh filename="file://$(find kortex_description)/gen3_arm/meshes/half_arm_1_link.dae" />
         </geometry>
       </collision>
@@ -181,14 +164,14 @@
         <origin xyz="0 0 0" rpy="0 0 0" />
         <geometry>
-          <mesh filename="file://$(find kortex_description)/arms/gen3/${dof}dof/meshes/half_arm_2_link.dae" />
-        </geometry>
-        <material name="">
-          <color rgba="0.75294 0.75294 0.75294 1" />
-        </material>
-      </visual>
-      <collision>
-        <origin xyz="0 0 0" rpy="0 0 0" />
-        <geometry>
-          <mesh filename="file://$(find kortex_description)/arms/gen3/${dof}dof/meshes/half_arm_2_link.dae" />
+          <mesh filename="file://$(find kortex_description)/gen3_arm/meshes/half_arm_2_link.dae" />
+        </geometry>
+        <material name="">
+          <color rgba="0.75294 0.75294 0.75294 1" />
+        </material>
+      </visual>
+      <collision>
+        <origin xyz="0 0 0" rpy="0 0 0" />
+        <geometry>
+          <mesh filename="file://$(find kortex_description)/gen3_arm/meshes/half_arm_2_link.dae" />
         </geometry>
       </collision>
@@ -237,14 +220,14 @@
         <origin xyz="0 0 0" rpy="0 0 0" />
         <geometry>
-          <mesh filename="file://$(find kortex_description)/arms/gen3/${dof}dof/meshes/forearm_link.dae" />
-        </geometry>
-        <material name="">
-          <color rgba="0.75294 0.75294 0.75294 1" />
-        </material>
-      </visual>
-      <collision>
-        <origin xyz="0 0 0" rpy="0 0 0" />
-        <geometry>
-          <mesh filename="file://$(find kortex_description)/arms/gen3/${dof}dof/meshes/forearm_link.dae" />
+          <mesh filename="file://$(find kortex_description)/gen3_arm/meshes/forearm_link.dae" />
+        </geometry>
+        <material name="">
+          <color rgba="0.75294 0.75294 0.75294 1" />
+        </material>
+      </visual>
+      <collision>
+        <origin xyz="0 0 0" rpy="0 0 0" />
+        <geometry>
+          <mesh filename="file://$(find kortex_description)/gen3_arm/meshes/forearm_link.dae" />
         </geometry>
       </collision>
@@ -271,14 +254,14 @@
         <origin xyz="0 0 0" rpy="0 0 0" />
         <geometry>
-          <mesh filename="file://$(find kortex_description)/arms/gen3/${dof}dof/meshes/spherical_wrist_1_link.dae" />
-        </geometry>
-        <material name="">
-          <color rgba="0.75294 0.75294 0.75294 1" />
-        </material>
-      </visual>
-      <collision>
-        <origin xyz="0 0 0" rpy="0 0 0" />
-        <geometry>
-          <mesh filename="file://$(find kortex_description)/arms/gen3/${dof}dof/meshes/spherical_wrist_1_link.dae" />
+          <mesh filename="file://$(find kortex_description)/gen3_arm/meshes/spherical_wrist_1_link.dae" />
+        </geometry>
+        <material name="">
+          <color rgba="0.75294 0.75294 0.75294 1" />
+        </material>
+      </visual>
+      <collision>
+        <origin xyz="0 0 0" rpy="0 0 0" />
+        <geometry>
+          <mesh filename="file://$(find kortex_description)/gen3_arm/meshes/spherical_wrist_1_link.dae" />
         </geometry>
       </collision>
@@ -327,14 +310,14 @@
         <origin xyz="0 0 0" rpy="0 0 0" />
         <geometry>
-          <mesh filename="file://$(find kortex_description)/arms/gen3/${dof}dof/meshes/spherical_wrist_2_link.dae" />
-        </geometry>
-        <material name="">
-          <color rgba="0.75294 0.75294 0.75294 1" />
-        </material>
-      </visual>
-      <collision>
-        <origin xyz="0 0 0" rpy="0 0 0" />
-        <geometry>
-          <mesh filename="file://$(find kortex_description)/arms/gen3/${dof}dof/meshes/spherical_wrist_2_link.dae" />
+          <mesh filename="file://$(find kortex_description)/gen3_arm/meshes/spherical_wrist_2_link.dae" />
+        </geometry>
+        <material name="">
+          <color rgba="0.75294 0.75294 0.75294 1" />
+        </material>
+      </visual>
+      <collision>
+        <origin xyz="0 0 0" rpy="0 0 0" />
+        <geometry>
+          <mesh filename="file://$(find kortex_description)/gen3_arm/meshes/spherical_wrist_2_link.dae" />
         </geometry>
       </collision>
@@ -362,14 +345,14 @@
         <origin xyz="0 0 0" rpy="0 0 0" />
         <geometry>
-          <mesh filename="file://$(find kortex_description)/arms/gen3/${dof}dof/meshes/bracelet_with_vision_link.dae" />
-        </geometry>
-        <material name="">
-          <color rgba="0.75294 0.75294 0.75294 1" />
-        </material>
-      </visual>
-      <collision>
-        <origin xyz="0 0 0" rpy="0 0 0" />
-        <geometry>
-          <mesh filename="file://$(find kortex_description)/arms/gen3/${dof}dof/meshes/bracelet_with_vision_link.dae" />
+          <mesh filename="file://$(find kortex_description)/gen3_arm/meshes/bracelet_with_vision_link.dae" />
+        </geometry>
+        <material name="">
+          <color rgba="0.75294 0.75294 0.75294 1" />
+        </material>
+      </visual>
+      <collision>
+        <origin xyz="0 0 0" rpy="0 0 0" />
+        <geometry>
+          <mesh filename="file://$(find kortex_description)/gen3_arm/meshes/bracelet_with_vision_link.dae" />
         </geometry>
       </collision>
@@ -386,14 +369,14 @@
         <origin xyz="0 0 0" rpy="0 0 0" />
         <geometry>
-          <mesh filename="file://$(find kortex_description)/arms/gen3/${dof}dof/meshes/bracelet_no_vision_link.dae" />
-        </geometry>
-        <material name="">
-          <color rgba="0.75294 0.75294 0.75294 1" />
-        </material>
-      </visual>
-      <collision>
-        <origin xyz="0 0 0" rpy="0 0 0" />
-        <geometry>
-          <mesh filename="file://$(find kortex_description)/arms/gen3/${dof}dof/meshes/bracelet_no_vision_link.dae" />
+          <mesh filename="file://$(find kortex_description)/gen3_arm/meshes/bracelet_no_vision_link.dae" />
+        </geometry>
+        <material name="">
+          <color rgba="0.75294 0.75294 0.75294 1" />
+        </material>
+      </visual>
+      <collision>
+        <origin xyz="0 0 0" rpy="0 0 0" />
+        <geometry>
+          <mesh filename="file://$(find kortex_description)/gen3_arm/meshes/bracelet_no_vision_link.dae" />
         </geometry>
       </collision>
@@ -447,26 +430,4 @@
     </joint>
     <xacro:if value="${vision}">
-      <!-- sim camera needs to be rotated which might not apply to built in vision module -->
-      <xacro:if value="${sim_ignition}">
-        <link name="${prefix}camera_link" />
-        <joint name="${prefix}camera_module" type="fixed">
-          <origin xyz="0 0.05639 0.01305" rpy="0 ${-PI/2} ${-PI/2}" />
-          <parent link="${prefix}end_effector_link" />
-          <child  link="${prefix}camera_link" />
-        </joint>
-        <link name="${prefix}camera_depth_frame" />
-        <joint name="${prefix}depth_module" type="fixed">
-          <origin xyz="0.0275 0.066 0.01305" rpy="0 ${-PI/2} ${-PI/2}" />
-          <parent link="${prefix}end_effector_link" />
-          <child  link="${prefix}camera_depth_frame" />
-        </joint>
-        <link name="${prefix}camera_color_frame" />
-        <joint name="${prefix}color_module" type="fixed">
-          <origin xyz="0 0.05639 0.01305" rpy="0 ${-PI/2} ${-PI/2}" />
-          <parent link="${prefix}end_effector_link" />
-          <child  link="${prefix}camera_color_frame" />
-        </joint>
-      </xacro:if>
-      <xacro:unless value="${sim_ignition}">
         <link name="${prefix}camera_link" />
         <joint name="${prefix}camera_module" type="fixed">
@@ -487,5 +448,4 @@
           <child  link="${prefix}camera_color_frame" />
         </joint>
-      </xacro:unless>
     </xacro:if>
   </xacro:macro>

File: kortex_description/gripper_robotiq_2f_85/urdf/robotiq_2f_85_macro.xacro (robot description, xacro)
@@ -2,19 +2,14 @@
 <robot name="robotiq_2f_85_model" xmlns:xacro="http://ros.org/wiki/xacro">
   <xacro:macro name="load_gripper" params="
-    parent
-    prefix
-    use_fake_hardware:=false
-    fake_sensor_commands:=false
-    sim_ignition:=false
-    sim_isaac:=false
-    isaac_joint_commands:=/isaac_joint_commands
-    isaac_joint_states:=/isaac_joint_states
+    parent:=end_effector_link
+    prefix:=""
     use_internal_bus_gripper_comm:=false
-    com_port:=/dev/ttyUSB0
-    moveit_active:=false">
+    com_port:=/dev/ttyUSB0">
     <xacro:include filename="$(find robotiq_description)/urdf/robotiq_2f_85_macro.urdf.xacro" />
     <!-- Hardware talks directly to the gripper so we don't need ros2_control unless we are simulating -->
-    <xacro:property name="include_ros2_control" value="false"/>
-    <xacro:if value="${sim_ignition or sim_isaac or use_fake_hardware or not use_internal_bus_gripper_comm}">
+    <xacro:if value="${use_internal_bus_gripper_comm}">
+      <xacro:property name="include_ros2_control" value="false"/>
+    </xacro:if>
+    <xacro:if value="${not use_internal_bus_gripper_comm}">
       <xacro:property name="include_ros2_control" value="true"/>
     </xacro:if>
@@ -24,11 +19,5 @@
         parent="${parent}"
         include_ros2_control="${include_ros2_control}"
-        com_port="${com_port}"
-        use_fake_hardware="${use_fake_hardware}"
-        fake_sensor_commands="${fake_sensor_commands}"
-        sim_ignition="${sim_ignition}"
-        sim_isaac="${sim_isaac}"
-        isaac_joint_commands="${isaac_joint_commands}"
-        isaac_joint_states="${isaac_joint_states}">
+        com_port="${com_port}">
         <origin xyz="0 0 0" rpy="0 0 0" />
     </xacro:robotiq_gripper>

File: kortex_description/robots/gen3.xacro (robot description, xacro)
@@ -3,8 +3,7 @@
     <!-- Arguments -->
     <xacro:arg name="arm" default="gen3" />
-    <xacro:arg name="dof" default="" />
     <xacro:arg name="vision" default="false" />
     <xacro:arg name="parent" default="world" />
-    <xacro:arg name="robot_ip" default="192.168.11.11" />
+    <xacro:arg name="robot_ip" default="192.168.1.10" />
     <xacro:arg name="username" default="admin" />
     <xacro:arg name="password" default="admin" />
@@ -17,17 +16,8 @@
     <xacro:arg name="gripper_max_velocity" default="100.0" />
     <xacro:arg name="gripper_max_force" default="100.0" />
-    <xacro:arg name="sim_gazebo" default="false" />
-    <xacro:arg name="sim_ignition" default="false" />
-    <xacro:arg name="sim_isaac" default="false" />
-    <xacro:arg name="prefix" default="" />
-    <xacro:arg name="use_fake_hardware" default="false" />
-    <xacro:arg name="fake_sensor_commands" default="false" />
     <xacro:arg name="use_internal_bus_gripper_comm" default="false" />
     <xacro:arg name="use_external_cable" default="false" />
     <xacro:arg name="initial_positions" default="${dict(joint_1=0.0,joint_2=0.0,joint_3=0.0,joint_4=0.0,joint_5=0.0,joint_6=0.0,joint_7=0.0)}"/>
-    <xacro:arg name="moveit_active" default="false" />
     <xacro:arg name="gripper_com_port" default="/dev/ttyUSB0" />
-    <xacro:arg name="isaac_joint_commands" default="/isaac_joint_commands" />
-    <xacro:arg name="isaac_joint_states" default="/isaac_joint_states" />
     <!-- Define world link -->
     <link name="world" />
@@ -37,5 +27,4 @@
     <xacro:load_arm
       parent="${parent}"
-      dof="${dof}"
       vision="${vision}"
       robot_ip="${robot_ip}"
@@ -46,28 +35,19 @@
       session_inactivity_timeout_ms="${session_inactivity_timeout_ms}"
       connection_inactivity_timeout_ms="${connection_inactivity_timeout_ms}"
-      prefix="${prefix}"
       use_internal_bus_gripper_comm="${use_internal_bus_gripper_comm}"
-      use_fake_hardware="${use_fake_hardware}"
-      fake_sensor_commands="${fake_sensor_commands}"
-      sim_gazebo="${sim_gazebo}"
-      sim_ignition="${sim_ignition}"
-      sim_isaac="${sim_isaac}"
-      isaac_joint_commands="${isaac_joint_commands}"
-      isaac_joint_states="${isaac_joint_states}"
       gripper_joint_name="${gripper_joint_name}"
       gripper_max_velocity="${gripper_max_velocity}"
       gripper_max_force="${gripper_max_force}"
       use_external_cable="${use_external_cable}"
-      initial_positions="${initial_positions}"
-      moveit_active="${moveit_active}">
+      initial_positions="${initial_positions}">
       <origin xyz="0 0 0" rpy="0 0 0" />  <!-- position the robotic arm in the world -->
     </xacro:load_arm>
     <!-- If no gripper, define tool frame here -->
     <xacro:if value="${not gripper}">
-      <link name="${prefix}tool_frame"/>
-      <joint name="${prefix}tool_frame_joint" type="fixed">
+      <link name="tool_frame"/>
+      <joint name="tool_frame_joint" type="fixed">
         <origin xyz="0 0 0" rpy="0 0 0" />
-        <parent link="${prefix}${last_arm_link}" />
-        <child link="${prefix}tool_frame" />
+        <parent link="${last_arm_link}" />
+        <child link="tool_frame" />
         <axis xyz="0 0 0" />
       </joint>
@@ -76,17 +56,9 @@
     <xacro:unless value="${not gripper}">
       <xacro:include filename="$(find kortex_description)/gripper_robotiq_2f_85/urdf/${gripper}_macro.xacro" />
-      <!-- last_arm_link is defined in "$(find kortex_description)/arms/${arm}/urdf/${arm}_macro.xacro" -->
+      <!-- last_arm_link is defined in "$(find kortex_description)/gen3_arm/urdf/${arm}_macro.xacro" -->
       <xacro:load_gripper
-        parent="${prefix}${last_arm_link}"
-        prefix="${prefix}"
-        use_fake_hardware="${use_fake_hardware}"
-        fake_sensor_commands="${fake_sensor_commands}"
-        sim_ignition="${sim_ignition}"
-        sim_isaac="${sim_isaac}"
-        isaac_joint_commands="${isaac_joint_commands}"
-        isaac_joint_states="${isaac_joint_states}"
+        parent="${last_arm_link}"
         com_port="${gripper_com_port}"
-        use_internal_bus_gripper_comm="${use_internal_bus_gripper_comm}"
-        moveit_active="${moveit_active}"/>
+        use_internal_bus_gripper_comm="${use_internal_bus_gripper_comm}"/>
     </xacro:unless>
   </xacro:macro>
