Commit message: Rectified minor issues with some .xacro files in the kortex_description package

File: kortex_description/gen3_arm/urdf/gen3_macro.xacro (robot description, xacro)
@@ -7,5 +7,5 @@
     parent:=world
     vision:=false
-    prefix:=""
+    prefix
     *origin
     robot_ip:=192.168.1.10
@@ -17,4 +17,5 @@
     connection_inactivity_timeout_ms:=2000
     use_internal_bus_gripper_comm:=false
+    tf_prefix
     gripper_joint_name:=finger_joint
     gripper_max_velocity:=100
@@ -35,4 +36,5 @@
       connection_inactivity_timeout_ms="${connection_inactivity_timeout_ms}"
       use_internal_bus_gripper_comm="${use_internal_bus_gripper_comm}"
+      tf_prefix="${tf_prefix}"
       gripper_max_velocity="${gripper_max_velocity}"
       gripper_max_force="${gripper_max_force}"

File: kortex_description/gripper_robotiq_2f_85/urdf/robotiq_2f_85_macro.xacro (robot description, xacro)
@@ -3,5 +3,5 @@
   <xacro:macro name="load_gripper" params="
     parent:=end_effector_link
-    prefix:=""
+    prefix
     use_internal_bus_gripper_comm:=false
     com_port:=/dev/ttyUSB0">

File: kortex_description/robots/gen3.xacro (robot description, xacro)
@@ -3,4 +3,5 @@
     <!-- Arguments -->
     <xacro:arg name="arm" default="gen3" />
+    <xacro:arg name="prefix" default="" />
     <xacro:arg name="vision" default="false" />
     <xacro:arg name="parent" default="world" />
@@ -17,32 +18,35 @@
     <xacro:arg name="gripper_max_force" default="100.0" />
     <xacro:arg name="use_internal_bus_gripper_comm" default="false" />
+    <xacro:arg name="tf_prefix" default="" />
     <xacro:arg name="use_external_cable" default="false" />
-    <xacro:arg name="initial_positions" default="${dict(joint_1=0.0,joint_2=0.0,joint_3=0.0,joint_4=0.0,joint_5=0.0,joint_6=0.0,joint_7=0.0)}"/>
     <xacro:arg name="gripper_com_port" default="/dev/ttyUSB0" />
     <!-- Define world link -->
     <link name="world" />
     <!-- Include and load arm macro files -->
-    <xacro:include filename="$(find kortex_description)/gen3_arm/urdf/${arm}_macro.xacro" />
+    <xacro:include filename="$(find kortex_description)/gen3_arm/urdf/gen3_macro.xacro" />
     <!-- Load the arm -->
     <xacro:load_arm
-      parent="${parent}"
-      vision="${vision}"
-      robot_ip="${robot_ip}"
-      username="${username}"
-      password="${password}"
-      port="${port}"
-      port_realtime="${port_realtime}"
-      session_inactivity_timeout_ms="${session_inactivity_timeout_ms}"
-      connection_inactivity_timeout_ms="${connection_inactivity_timeout_ms}"
-      use_internal_bus_gripper_comm="${use_internal_bus_gripper_comm}"
-      gripper_joint_name="${gripper_joint_name}"
-      gripper_max_velocity="${gripper_max_velocity}"
-      gripper_max_force="${gripper_max_force}"
-      use_external_cable="${use_external_cable}"
-      initial_positions="${initial_positions}">
+      prefix="$(arg prefix)"
+      parent="$(arg parent)"
+      vision="$(arg vision)"
+      robot_ip="$(arg robot_ip)"
+      username="$(arg username)"
+      password="$(arg password)"
+      port="$(arg port)"
+      port_realtime="$(arg port_realtime)"
+      session_inactivity_timeout_ms="$(arg session_inactivity_timeout_ms)"
+      connection_inactivity_timeout_ms="$(arg connection_inactivity_timeout_ms)"
+      use_internal_bus_gripper_comm="$(arg use_internal_bus_gripper_comm)"
+      tf_prefix="$(arg tf_prefix)"
+      gripper_joint_name="$(arg gripper_joint_name)"
+      gripper_max_velocity="$(arg gripper_max_velocity)"
+      gripper_max_force="$(arg gripper_max_force)"
+      use_external_cable="$(arg use_external_cable)">
       <origin xyz="0 0 0" rpy="0 0 0" />  <!-- position the robotic arm in the world -->
     </xacro:load_arm>
+    <!-- Convert the argument to a Xacro property with a different name -->
+    <xacro:property name="gripper_arg" value="$(arg gripper)" />
     <!-- If no gripper, define tool frame here -->
-    <xacro:if value="${not gripper}">
+    <xacro:if value="${gripper_arg == ''}">
       <link name="tool_frame"/>
       <joint name="tool_frame_joint" type="fixed">
@@ -54,12 +58,13 @@
     </xacro:if>
     <!-- Include and load the gripper if defined -->
-    <xacro:unless value="${not gripper}">
-      <xacro:include filename="$(find kortex_description)/gripper_robotiq_2f_85/urdf/${gripper}_macro.xacro" />
+    <xacro:unless value="${gripper_arg == ''}">
+      <xacro:include filename="$(find kortex_description)/gripper_robotiq_2f_85/urdf/robotiq_2f_85_macro.xacro" />
       <!-- last_arm_link is defined in "$(find kortex_description)/gen3_arm/urdf/${arm}_macro.xacro" -->
       <xacro:load_gripper
-        parent="${last_arm_link}"
-        com_port="${gripper_com_port}"
-        use_internal_bus_gripper_comm="${use_internal_bus_gripper_comm}"/>
+        parent="$(arg prefix)${last_arm_link}"
+        prefix="$(arg prefix)"
+        com_port="$(arg gripper_com_port)"
+        use_internal_bus_gripper_comm="$(arg use_internal_bus_gripper_comm)">
+      </xacro:load_gripper>
     </xacro:unless>
-  </xacro:macro>
 </robot>
